File: Project3.kicad_sch (KiCad schematic)
At the start: 0 parts

Commit message: THT Footprint assigned
Parts:
- added BT1, BT2: Battery_Cell, Battery:BatteryHolder_Seiko_MS621F, symbol Device:Battery_Cell
- added D1, D2: LED, LED_THT:LED_D3.0mm, symbol Device:LED
- added R1, R2: R, Resistor_THT:R_Axial_DIN0207_L6.3mm_D2.5mm_P10.16mm_Horizontal, symbol Device:R
- added SW1: SW_Push_Open, Button_Switch_THT:SW_TH_Tactile_Omron_B3F-106x, symbol Switch:SW_Push_Open
Connections:
- new net: BT1.1 (+), BT2.1 (+), R1.2, R2.2
- new net: BT1.2 (-), BT2.2 (-), SW1.2 (B)
- new net: D1.1 (K), D2.1 (K), SW1.1 (A)
- new net: D2.2 (A), R2.1
- new net: D1.2 (A), R1.1
