File: _autosave-Project3.kicad_sch (KiCad schematic)
At the start: 7 parts, among them SW1 SW_Push_Open

Commit message: Updated PCB and schematic
Parts:
- BT1, BT2: footprint Battery:BatteryHolder_Seiko_MS621F -> Connector_Molex:Molex_KK-254_AE-6410-02A_1x02_P2.54mm_Vertical
Changed lines of the file:
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@@
 			)
 		)
-		(property "Footprint" "Battery:BatteryHolder_Seiko_MS621F"
+		(property "Footprint" "Connector_Molex:Molex_KK-254_AE-6410-02A_1x02_P2.54mm_Vertical"
 			(at 175.26 98.044 90)
 			(effects
@@
 			)
 		)
-		(property "Footprint" "Battery:BatteryHolder_Seiko_MS621F"
+		(property "Footprint" "Connector_Molex:Molex_KK-254_AE-6410-02A_1x02_P2.54mm_Vertical"
 			(at 154.94 98.044 90)
 			(effects
